Commit message: more work on navigation node

File: src/furiguide_description/urdf/furiguide.xacro (robot description, xacro)
@@ -117,4 +117,89 @@
 <wheel lr="left" parent="chassis" translateY="0.5"/>
 <wheel lr="right" parent="chassis" translateY="-0.5"/>
+<!-- Camera -->
+<joint name="camera_joint" type="fixed">
+  <axis xyz="0 1 0" />
+  <origin xyz="0 0 0" rpy="0 0 0" />
+  <parent link="chassis" />
+  <child link="camera_link" />
+</joint>
+<link name="camera_link">
+  <inertial>
+    <mass value="1e-5" />
+    <origin xyz="0 0 0" rpy="0 0 0" />
+    <inertia ixx="1e-6" ixy="0" ixz="0" iyy="1e-6" iyz="0" izz="1e-6" />
+  </inertial>
+  <collision>
+    <origin xyz="0 0 0.05" rpy="0 0 0" />
+    <geometry>
+      <box size="0.01 0.01 0.01" />
+    </geometry>
+  </collision>
+  <visual>
+    <origin xyz="0 0 0.05" rpy="0 0 0" />
+    <geometry>
+      <box size="0.01 0.01 0.01" />
+    </geometry>
+  </visual>
+</link>
+<!-- generate an optical frame http://www.ros.org/reps/rep-0103.html#suffix-frames
+    so that ros and opencv can operate on the camera frame correctly -->
+<joint name="camera_optical_joint" type="fixed">
+  <!-- these values have to be these values otherwise the gazebo camera image
+      won't be aligned properly with the frame it is supposedly originating from -->
+  <origin xyz="0 0 0" rpy="${-M_PI/2} 0 ${-M_PI/2}"/>
+  <parent link="camera_link"/>
+  <child link="camera_link_optical"/>
+</joint>
+<link name="camera_link_optical">
+</link>
+<gazebo reference="camera_link">
+  <sensor type="camera" name="camera1">
+    <update_rate>10.0</update_rate>
+    <camera name="head">
+      <horizontal_fov>1.3962634</horizontal_fov>
+      <image>
+        <width>800</width>
+        <height>800</height>
+        <format>R8G8B8</format>
+      </image>
+      <clip>
+        <near>0.02</near>
+        <far>300</far>
+      </clip>
+      <noise>
+        <type>gaussian</type>
+        <!-- Noise is sampled independently per pixel on each frame.
+             That pixel's noise value is added to each of its color
+             channels, which at that point lie in the range [0,1]. -->
+        <mean>0.0</mean>
+        <stddev>0.007</stddev>
+      </noise>
+    </camera>
+    <plugin name="camera_controller" filename="libgazebo_ros_camera.so">
+      <robotNamespace>/furiguide</robotNamespace>
+      <alwaysOn>true</alwaysOn>
+      <updateRate>0.0</updateRate>
+      <cameraName>camera1</cameraName>
+      <imageTopicName>image_raw</imageTopicName>
+      <cameraInfoTopicName>camera_info</cameraInfoTopicName>
+      <frameName>camera_link_optical</frameName>
+      <!-- setting hackBaseline to anything but 0.0 will cause a misalignment
+      between the gazebo sensor image and the frame it is supposed to
+      be attached to -->
+      <hackBaseline>0.0</hackBaseline>
+      <distortionK1>0.0</distortionK1>
+      <distortionK2>0.0</distortionK2>
+      <distortionK3>0.0</distortionK3>
+      <distortionT1>0.0</distortionT1>
+      <distortionT2>0.0</distortionT2>
+      <CxPrime>0</CxPrime>
+      <Cx>0.0</Cx>
+      <Cy>0.0</Cy>
+      <focalLength>0.0</focalLength>
+    </plugin>
+  </sensor>
+  <material>Gazebo/Green</material>
+</gazebo>
 <!-- Gazebo Specific Configuration -->
 <gazebo>

Commit message: improved gazebo simulation and rviz support

File: src/furiguide_description/urdf/furiguide.xacro (robot description, xacro)
@@ -120,5 +120,5 @@
 <joint name="camera_joint" type="fixed">
   <axis xyz="0 1 0" />
-  <origin xyz="0 0 0" rpy="0 0 0" />
+  <origin xyz="0.12 0 0.2" rpy="0 0 0" />
   <parent link="chassis" />
   <child link="camera_link" />
@@ -131,5 +131,5 @@
   </inertial>
   <collision>
-    <origin xyz="0 0 0.05" rpy="0 0 0" />
+    <origin xyz="0 0 0.05" rpy="0 0.4 0" />
     <geometry>
       <box size="0.01 0.01 0.01" />
@@ -137,5 +137,5 @@
   </collision>
   <visual>
-    <origin xyz="0 0 0.05" rpy="0 0 0" />
+    <origin xyz="0 0 0.05" rpy="0 0.4 0" />
     <geometry>
       <box size="0.01 0.01 0.01" />
@@ -156,10 +156,10 @@
 <gazebo reference="camera_link">
   <sensor type="camera" name="camera1">
-    <update_rate>10.0</update_rate>
+    <update_rate>30.0</update_rate>
     <camera name="head">
       <horizontal_fov>1.3962634</horizontal_fov>
       <image>
         <width>800</width>
-        <height>800</height>
+        <height>600</height>
         <format>R8G8B8</format>
       </image>
@@ -178,5 +178,4 @@
     </camera>
     <plugin name="camera_controller" filename="libgazebo_ros_camera.so">
-      <robotNamespace>/furiguide</robotNamespace>
       <alwaysOn>true</alwaysOn>
       <updateRate>0.0</updateRate>

Commit message: support two cameras in launch files

File: src/furiguide_description/urdf/furiguide.xacro (robot description, xacro)
@@ -143,17 +143,43 @@
   </visual>
 </link>
+<!-- Rear Camera -->
+<joint name="camera__rear_joint" type="fixed">
+  <axis xyz="0 1 0" />
+  <origin xyz="-0.12 0 0.2" rpy="0 0 ${M_PI}" />
+  <parent link="chassis" />
+  <child link="camera_rear_link" />
+</joint>
+<link name="camera_rear_link">
+  <inertial>
+    <mass value="1e-5" />
+    <origin xyz="0 0 0" rpy="0 0 0" />
+    <inertia ixx="1e-6" ixy="0" ixz="0" iyy="1e-6" iyz="0" izz="1e-6" />
+  </inertial>
+  <collision>
+    <origin xyz="0 0 0.05" rpy="0 -0.4 0" />
+    <geometry>
+      <box size="0.01 0.01 0.01" />
+    </geometry>
+  </collision>
+  <visual>
+    <origin xyz="0 0 0.05" rpy="0 -0.4 0" />
+    <geometry>
+      <box size="0.01 0.01 0.01" />
+    </geometry>
+  </visual>
+</link>
 <!-- generate an optical frame http://www.ros.org/reps/rep-0103.html#suffix-frames
     so that ros and opencv can operate on the camera frame correctly -->
-<joint name="camera_optical_joint" type="fixed">
+<joint name="camera_rear_optical_joint" type="fixed">
   <!-- these values have to be these values otherwise the gazebo camera image
       won't be aligned properly with the frame it is supposedly originating from -->
   <origin xyz="0 0 0" rpy="${-M_PI/2} 0 ${-M_PI/2}"/>
-  <parent link="camera_link"/>
-  <child link="camera_link_optical"/>
+  <parent link="camera_rear_link"/>
+  <child link="camera_rear_link_optical"/>
 </joint>
-<link name="camera_link_optical">
-</link>
-<gazebo reference="camera_link">
-  <sensor type="camera" name="camera1">
+<link name="camera_rear_link_optical">
+</link>
+<gazebo reference="camera_rear_link">
+  <sensor type="camera" name="camera_rear">
     <update_rate>30.0</update_rate>
     <camera name="head">
@@ -180,5 +206,63 @@
       <alwaysOn>true</alwaysOn>
       <updateRate>0.0</updateRate>
-      <cameraName>camera1</cameraName>
+      <cameraName>camera_rear</cameraName>
+      <imageTopicName>image_raw</imageTopicName>
+      <cameraInfoTopicName>camera_info</cameraInfoTopicName>
+      <frameName>camera_rear_link_optical</frameName>
+      <!-- setting hackBaseline to anything but 0.0 will cause a misalignment
+      between the gazebo sensor image and the frame it is supposed to
+      be attached to -->
+      <hackBaseline>0.0</hackBaseline>
+      <distortionK1>0.0</distortionK1>
+      <distortionK2>0.0</distortionK2>
+      <distortionK3>0.0</distortionK3>
+      <distortionT1>0.0</distortionT1>
+      <distortionT2>0.0</distortionT2>
+      <CxPrime>0</CxPrime>
+      <Cx>0.0</Cx>
+      <Cy>0.0</Cy>
+      <focalLength>0.0</focalLength>
+    </plugin>
+  </sensor>
+  <material>Gazebo/Blue</material>
+</gazebo>
+<!-- generate an optical frame http://www.ros.org/reps/rep-0103.html#suffix-frames
+    so that ros and opencv can operate on the camera frame correctly -->
+<joint name="camera_optical_joint" type="fixed">
+  <!-- these values have to be these values otherwise the gazebo camera image
+      won't be aligned properly with the frame it is supposedly originating from -->
+  <origin xyz="0 0 0" rpy="${-M_PI/2} 0 ${-M_PI/2}"/>
+  <parent link="camera_link"/>
+  <child link="camera_link_optical"/>
+</joint>
+<link name="camera_link_optical">
+</link>
+<gazebo reference="camera_link">
+  <sensor type="camera" name="camera_front">
+    <update_rate>30.0</update_rate>
+    <camera name="head">
+      <horizontal_fov>1.3962634</horizontal_fov>
+      <image>
+        <width>800</width>
+        <height>600</height>
+        <format>R8G8B8</format>
+      </image>
+      <clip>
+        <near>0.02</near>
+        <far>300</far>
+      </clip>
+      <noise>
+        <type>gaussian</type>
+        <!-- Noise is sampled independently per pixel on each frame.
+             That pixel's noise value is added to each of its color
+             channels, which at that point lie in the range [0,1]. -->
+        <mean>0.0</mean>
+        <stddev>0.007</stddev>
+      </noise>
+    </camera>
+    <plugin name="camera_controller" filename="libgazebo_ros_camera.so">
+      <alwaysOn>true</alwaysOn>
+      <updateRate>0.0</updateRate>
+      <cameraName>camera_front</cameraName>
       <imageTopicName>image_raw</imageTopicName>
       <cameraInfoTopicName>camera_info</cameraInfoTopicName>

Commit message: add LiDAR to furiguide model

File: src/furiguide_description/urdf/furiguide.xacro (robot description, xacro)
@@ -48,4 +48,10 @@
   </visual>
 </xacro:macro>
+<link name='base_link'/>
+<joint name="base_joint" type="fixed">
+  <origin xyz="0 0 0.0102" rpy="0 0 0" />
+  <parent link="base_link"/>
+  <child link="chassis" />
+</joint>
 <link name='chassis'>
   <pose>0 0 0.1 0 0 0</pose>
@@ -72,4 +78,32 @@
   <caster fb="front" translateX="-0.15" />
   <caster fb="rear" translateX="0.15" />
+</link>
+<joint name="upper_joint" type="fixed">
+  <origin xyz="0 0 0.25" rpy="0 0 0" />
+  <parent link="base_link" />
+  <child link="upper_chassis" />
+</joint>
+<link name='upper_chassis'>
+  <pose>0 0 0.0 0 0 0</pose>
+  <inertial>
+    <mass value="${base_mass}"/>
+    <origin xyz="0.0 0 0.0" rpy="0 0 0"/>
+    <inertia
+      ixx="0.1" ixy="0" ixz="0"
+      iyy="0.1" iyz="0"
+      izz="0.1"
+    />
+  </inertial>
+  <collision name='collision'>
+    <geometry>
+      <cylinder length="${base_height}" radius="${base_radius}"/>
+    </geometry>
+  </collision>
+  <visual name='chassis_visual'>
+    <origin xyz="0 0 0" rpy="0 0 0"/>
+    <geometry>
+      <cylinder length="${base_height}" radius="${base_radius}"/>
+    </geometry>
+  </visual>
 </link>
 <!-- Wheels -->
@@ -120,6 +154,6 @@
 <joint name="camera_joint" type="fixed">
   <axis xyz="0 1 0" />
-  <origin xyz="0.12 0 0.2" rpy="0 0 0" />
-  <parent link="chassis" />
+  <origin xyz="0.12 0 0" rpy="0 0 0" />
+  <parent link="upper_chassis" />
   <child link="camera_link" />
 </joint>
@@ -201,4 +235,64 @@
   <material>Gazebo/Green</material>
 </gazebo>
+<!-- LiDAR -->
+<link name="rplidar_link">
+  <inertial>
+    <mass value="1e-5" />
+    <origin xyz="0 0 0" rpy="0 0 0" />
+    <inertia ixx="1e-6" ixy="0" ixz="0" iyy="1e-6" iyz="0" izz="1e-6" />
+  </inertial>
+  <collision>
+    <origin xyz="0 0 0" rpy="0 0 0" />
+    <geometry>
+      <cylinder length="0.05" radius="0.05"/>
+    </geometry>
+  </collision>
+  <visual>
+    <origin xyz="0 0 0" rpy="0 0 0" />
+    <geometry>
+      <cylinder length="0.05" radius="0.05"/>
+    </geometry>
+  </visual>
+</link>
+<joint name="rplidar_joint" type="fixed">
+  <origin xyz="0 0 0.0102" rpy="0 0 0" />
+  <parent link="upper_chassis"/>
+  <child link="rplidar_link" />
+</joint>
+<gazebo reference="rplidar_link">
+  <sensor type="gpu_ray" name="head_hokuyo_sensor">
+    <pose>0 0 0 0 0 0</pose>
+    <visualize>false</visualize>
+    <update_rate>40</update_rate>
+    <ray>
+      <scan>
+        <horizontal>
+          <samples>720</samples>
+          <resolution>1</resolution>
+          <min_angle>-1.570796</min_angle>
+          <max_angle>1.570796</max_angle>
+        </horizontal>
+      </scan>
+      <range>
+        <min>0.10</min>
+        <max>30.0</max>
+        <resolution>0.01</resolution>
+      </range>
+      <noise>
+        <type>gaussian</type>
+        <!-- Noise parameters based on published spec for Hokuyo laser
+              achieving "+-30mm" accuracy at range < 10m.  A mean of 0.0m and
+              stddev of 0.01m will put 99.7% of samples within 0.03m of the true
+              reading. -->
+        <mean>0.0</mean>
+        <stddev>0.01</stddev>
+      </noise>
+    </ray>
+    <plugin name="gazebo_ros_head_hokuyo_controller" filename="libgazebo_ros_gpu_laser.so">
+      <topicName>/furiguide/laser/scan</topicName>
+      <frameName>rplidar_link</frameName>
+    </plugin>
+  </sensor>
+</gazebo>
 <!-- Gazebo Specific Configuration -->
 <gazebo>
@@ -215,5 +309,5 @@
     <odometryTopic>odom</odometryTopic>
     <odometryFrame>odom</odometryFrame>
-    <robotBaseFrame>chassis</robotBaseFrame>
+    <robotBaseFrame>base_link</robotBaseFrame>
   </plugin>
 </gazebo>

Commit message: Updated furiguide URDF model

File: src/furiguide_description/urdf/furiguide.xacro (robot description, xacro)
@@ -4,17 +4,25 @@
 <!-- Properties (MKS) -->
 <xacro:property name="M_PI" value="3.1415926535897931"/>
-<xacro:property name="base_height" value="0.02" />
+<xacro:property name="base_height" value="0.005"/>
+<xacro:property name="base_length" value="0.255" />
+<xacro:property name="base_width" value="0.28" />
 <xacro:property name="base_radius" value="0.15" />
 <xacro:property name="base_mass" value="5" />
-<xacro:property name="caster_height" value="0.08" />
-<xacro:property name="caster_radius" value="0.025" />
+<xacro:property name="base_separation" value="0.065" />
+<xacro:property name="caster_height" value="0.065" />
+<xacro:property name="caster_radius" value="0.005" />
+<xacro:property name="caster_offset" value="0.115" />
 <xacro:property name="caster_mass" value="0.5" />
 <xacro:property name="wheel_mass" value="0.25" />
-<xacro:property name="wheel_height" value="0.04" />
-<xacro:property name="wheel_radius" value="0.08" />
-<xacro:property name="wheel_separation" value="0.4" />
-<xacro:property name="base_x_origin_to_wheel_origin" value="0.25" />
-<xacro:property name="base_y_origin_to_wheel_origin" value="0.3" />
-<xacro:property name="base_z_origin_to_wheel_origin" value="0.0" />
+<xacro:property name="wheel_height" value="0.024" />
+<xacro:property name="wheel_radius" value="0.0425" />
+<xacro:property name="wheel_separation" value="0.3" />
+<xacro:property name="base_x_origin_to_wheel_origin" value="0.0" />
+<xacro:property name="base_y_origin_to_wheel_origin" value="${wheel_separation / 2}" />
+<xacro:property name="base_z_origin_to_wheel_origin" value="-0.025" />
+<!-- Sensor Dimensions -->
+<xacro:property name="lidar_base_separation" value="0.015" />
+<xacro:property name="lidar_height" value="0.04" />
+<xacro:property name="lidar_radius" value="0.0375" />
 <!-- Cylinder Inertia Macro (source: Kaustav5422) -->
 <xacro:macro name="cylinder_inertia" params="m r h">
@@ -24,29 +32,36 @@
 </xacro:macro>
 <!-- Caster -->
-<xacro:macro name="caster" params="fb translateX:=0 translateY:=0">
-  <collision name='${fb}_caster_collision'>
-    <origin xyz="${translateX} 0 -0.05" rpy="0 0 0"/>
-    <geometry>
-      <sphere radius="${caster_radius}"/>
-    </geometry>
-    <surface>
-      <friction>
-        <ode>
-          <mu>0</mu>
-          <mu2>0</mu2>
-          <slip1>1.0</slip1>
-          <slip2>1.0</slip2>
-        </ode>
-      </friction>
-    </surface>
-  </collision>
-  <visual name='${fb}_caster_visual'>
-    <origin xyz="${translateX} 0 -0.05" rpy="0 0 0"/>
-    <geometry>
-      <sphere radius="${caster_radius}"/>
-    </geometry>
-  </visual>
+<xacro:macro name="caster" params="fb translateX:=0">
+  <link name="${fb}_caster">
+    <collision name="${fb}_caster_collision">
+      <origin xyz="0 0 0" rpy="0 0 0"/>
+      <geometry>
+        <sphere radius="${caster_radius}"/>
+      </geometry>
+      <surface>
+        <friction>
+          <ode>
+            <mu>0</mu>
+            <mu2>0</mu2>
+            <slip1>1.0</slip1>
+            <slip2>1.0</slip2>
+          </ode>
+        </friction>
+      </surface>
+    </collision>
+    <visual name="${fb}_caster_visual">
+      <origin xyz="0 0 0" rpy="0 0 0"/>
+      <geometry>
+        <sphere radius="${caster_radius}"/>
+      </geometry>
+    </visual>
+  </link>
+  <joint name="${fb}_caster_fixed" type="fixed">
+    <origin xyz="${translateX} 0 -${caster_height}" rpy="0 0 0"/>
+    <parent link="chassis" />
+    <child link="${fb}_caster" />
+  </joint>
 </xacro:macro>
-<link name='base_link'/>
+<link name="base_link"/>
 <joint name="base_joint" type="fixed">
   <origin xyz="0 0 0.0102" rpy="0 0 0" />
@@ -54,5 +69,5 @@
   <child link="chassis" />
 </joint>
-<link name='chassis'>
+<link name="chassis">
   <pose>0 0 0.1 0 0 0</pose>
   <inertial>
@@ -65,24 +80,25 @@
     />
   </inertial>
-  <collision name='collision'>
-    <geometry>
-      <cylinder length="${base_height}" radius="${base_radius}"/>
+  <collision name="collision">
+    <origin xyz="0 0 0" rpy="0 0 0"/>
+    <geometry>
+      <box size="${base_width} ${base_length} ${base_height}" />
     </geometry>
   </collision>
-  <visual name='chassis_visual'>
+  <visual name="chassis_visual">
     <origin xyz="0 0 0" rpy="0 0 0"/>
     <geometry>
-      <cylinder length="${base_height}" radius="${base_radius}"/>
+      <box size="${base_width} ${base_length} ${base_height}" />
     </geometry>
   </visual>
-  <caster fb="front" translateX="-0.15" />
-  <caster fb="rear" translateX="0.15" />
-</link>
+</link>
+<caster fb="front" translateX="-0.15" />
+<caster fb="rear" translateX="0.15" />
 <joint name="upper_joint" type="fixed">
-  <origin xyz="0 0 0.25" rpy="0 0 0" />
+  <origin xyz="0 0 ${base_separation}" rpy="0 0 0" />
   <parent link="base_link" />
   <child link="upper_chassis" />
 </joint>
-<link name='upper_chassis'>
+<link name="upper_chassis">
   <pose>0 0 0.0 0 0 0</pose>
   <inertial>
@@ -95,13 +111,13 @@
     />
   </inertial>
-  <collision name='collision'>
-    <geometry>
-      <cylinder length="${base_height}" radius="${base_radius}"/>
+  <collision name="collision">
+    <geometry>
+      <box size="${base_length} ${base_width} ${base_height}" />
     </geometry>
   </collision>
-  <visual name='chassis_visual'>
+  <visual name="chassis_visual">
     <origin xyz="0 0 0" rpy="0 0 0"/>
     <geometry>
-      <cylinder length="${base_height}" radius="${base_radius}"/>
+      <box size="${base_length} ${base_width} ${base_height}" />
     </geometry>
   </visual>
@@ -138,5 +154,4 @@
   </gazebo>
   <joint type="continuous" name="${lr}_wheel_axle">
-    <child link="${lr}_wheel" />
     <origin xyz="${translateX * base_x_origin_to_wheel_origin}
                  ${translateY * base_y_origin_to_wheel_origin}
@@ -144,4 +159,5 @@
             rpy="0 0 0" />
     <parent link="${parent}" />
+    <child link="${lr}_wheel" />
     <axis xyz="0 1 0" rpy="0 0 0" />
     <limit effort="100" velocity="100" />
@@ -149,10 +165,10 @@
   </joint>
 </xacro:macro>
-<wheel lr="left" parent="chassis" translateY="0.5"/>
-<wheel lr="right" parent="chassis" translateY="-0.5"/>
+<wheel lr="left" parent="chassis" translateY="1"/>
+<wheel lr="right" parent="chassis" translateY="-1"/>
 <!-- Camera -->
 <joint name="camera_joint" type="fixed">
   <axis xyz="0 1 0" />
-  <origin xyz="0.12 0 0" rpy="0 0 0" />
+  <origin xyz="${base_length/2 - 0.021} 0 0.0125" rpy="0 0 ${M_PI/2}" />
   <parent link="upper_chassis" />
   <child link="camera_link" />
@@ -165,13 +181,13 @@
   </inertial>
   <collision>
-    <origin xyz="0 0 0.05" rpy="0 0.4 0" />
-    <geometry>
-      <box size="0.01 0.01 0.01" />
+    <origin xyz="0 0 0" rpy="0 0 0" />
+    <geometry>
+      <box size="0.09 0.025 0.025" />
     </geometry>
   </collision>
   <visual>
-    <origin xyz="0 0 0.05" rpy="0 0.4 0" />
-    <geometry>
-      <box size="0.01 0.01 0.01" />
+    <origin xyz="0 0 0" rpy="0 0 0" />
+    <geometry>
+      <box size="0.09 0.025 0.025" />
     </geometry>
   </visual>
@@ -188,17 +204,20 @@
 <link name="camera_link_optical">
 </link>
+<!-- Intel Realsense D435 Camera -->
 <gazebo reference="camera_link">
   <sensor type="camera" name="camera1">
-    <update_rate>30.0</update_rate>
+    <update_rate>60.0</update_rate>
     <camera name="head">
-      <horizontal_fov>1.3962634</horizontal_fov>
+      <!-- 69.4 x 42.5 degrees -->
+      <horizontal_fov>1.211258501</horizontal_fov>
+      <vertical_fov>0.741764932</vertical_fov>
       <image>
-        <width>800</width>
-        <height>600</height>
+        <width>1920</width>
+        <height>1080</height>
         <format>R8G8B8</format>
       </image>
       <clip>
-        <near>0.02</near>
-        <far>300</far>
+        <near>0.011</near>
+        <far>10</far>
       </clip>
       <noise>
@@ -245,5 +264,5 @@
     <origin xyz="0 0 0" rpy="0 0 0" />
     <geometry>
-      <cylinder length="0.05" radius="0.05"/>
+      <cylinder length="${lidar_height}" radius="${lidar_radius}"/>
     </geometry>
   </collision>
@@ -251,10 +270,10 @@
     <origin xyz="0 0 0" rpy="0 0 0" />
     <geometry>
-      <cylinder length="0.05" radius="0.05"/>
+      <cylinder length="${lidar_height}" radius="${lidar_radius}"/>
     </geometry>
   </visual>
 </link>
 <joint name="rplidar_joint" type="fixed">
-  <origin xyz="0 0 0.0102" rpy="0 0 0" />
+  <origin xyz="0 0 ${lidar_base_separation + lidar_height/2 + base_height}" rpy="0 0 0" />
   <parent link="upper_chassis"/>
   <child link="rplidar_link" />
