Commit message: fix furiguide model camera frame and caster height

File: src/furiguide_description/urdf/furiguide.xacro (robot description, xacro)
@@ -10,5 +10,5 @@
 <xacro:property name="base_mass" value="5" />
 <xacro:property name="base_separation" value="0.065" />
-<xacro:property name="caster_height" value="0.065" />
+<xacro:property name="caster_height" value="0.062" />
 <xacro:property name="caster_radius" value="0.005" />
 <xacro:property name="caster_offset" value="0.115" />
@@ -170,5 +170,5 @@
 <joint name="camera_joint" type="fixed">
   <axis xyz="0 1 0" />
-  <origin xyz="${base_length/2 - 0.021} 0 0.0125" rpy="0 0 ${M_PI/2}" />
+  <origin xyz="${base_length/2 - 0.021} 0 0.0125" rpy="0 0 0" />
   <parent link="upper_chassis" />
   <child link="camera_link" />
@@ -181,5 +181,5 @@
   </inertial>
   <collision>
-    <origin xyz="0 0 0" rpy="0 0 0" />
+    <origin xyz="0 0 0" rpy="0 0 ${M_PI/2}" />
     <geometry>
       <box size="0.09 0.025 0.025" />
@@ -187,5 +187,5 @@
   </collision>
   <visual>
-    <origin xyz="0 0 0" rpy="0 0 0" />
+    <origin xyz="0 0 0" rpy="0 0 ${M_PI/2}" />
     <geometry>
       <box size="0.09 0.025 0.025" />
@@ -198,5 +198,5 @@
   <!-- these values have to be these values otherwise the gazebo camera image
       won't be aligned properly with the frame it is supposedly originating from -->
-  <origin xyz="0 0 0" rpy="${-M_PI/2} 0 ${-M_PI/2}"/>
+  <origin xyz="0 0 0" rpy="-${M_PI/2} 0 -${M_PI/2}"/>
   <parent link="camera_link"/>
   <child link="camera_link_optical"/>
@@ -211,8 +211,7 @@
       <!-- 69.4 x 42.5 degrees -->
       <horizontal_fov>1.211258501</horizontal_fov>
-      <vertical_fov>0.741764932</vertical_fov>
       <image>
-        <width>1920</width>
-        <height>1080</height>
+        <width>1280</width>
+        <height>720</height>
         <format>R8G8B8</format>
       </image>

Commit message: rudimentiary Djikstra path planning
* more parameter and model tweaking

File: src/furiguide_description/urdf/furiguide.xacro (robot description, xacro)
@@ -8,14 +8,14 @@
 <xacro:property name="base_width" value="0.28" />
 <xacro:property name="base_radius" value="0.15" />
-<xacro:property name="base_mass" value="5" />
+<xacro:property name="base_mass" value="10" />
 <xacro:property name="base_separation" value="0.065" />
-<xacro:property name="caster_height" value="0.062" />
-<xacro:property name="caster_radius" value="0.005" />
+<xacro:property name="caster_height" value="0.04725" />
+<xacro:property name="caster_radius" value="0.020" />
 <xacro:property name="caster_offset" value="0.115" />
 <xacro:property name="caster_mass" value="0.5" />
-<xacro:property name="wheel_mass" value="0.25" />
-<xacro:property name="wheel_height" value="0.024" />
+<xacro:property name="wheel_mass" value="1.0" />
+<xacro:property name="wheel_height" value="0.05" />
 <xacro:property name="wheel_radius" value="0.0425" />
-<xacro:property name="wheel_separation" value="0.3" />
+<xacro:property name="wheel_separation" value="0.325" />
 <xacro:property name="base_x_origin_to_wheel_origin" value="0.0" />
 <xacro:property name="base_y_origin_to_wheel_origin" value="${wheel_separation / 2}" />
@@ -34,4 +34,13 @@
 <xacro:macro name="caster" params="fb translateX:=0">
   <link name="${fb}_caster">
+    <inertial>
+      <mass value="${wheel_mass}"/>
+      <origin xyz="0 0 0" />
+      <inertia
+        ixx="0.01" ixy="0" ixz="0"
+        iyy="0.01" iyz="0"
+        izz="0.01"
+      />
+    </inertial>
     <collision name="${fb}_caster_collision">
       <origin xyz="0 0 0" rpy="0 0 0"/>
@@ -72,5 +81,5 @@
   <pose>0 0 0.1 0 0 0</pose>
   <inertial>
-    <mass value="${base_mass}"/>
+    <mass value="${base_mass*0.75}"/>
     <origin xyz="0.0 0 0.1" rpy="0 0 0"/>
     <inertia
@@ -103,5 +112,5 @@
   <pose>0 0 0.0 0 0 0</pose>
   <inertial>
-    <mass value="${base_mass}"/>
+    <mass value="${base_mass*0.25}"/>
     <origin xyz="0.0 0 0.0" rpy="0 0 0"/>
     <inertia
@@ -146,6 +155,6 @@
   </link>
   <gazebo reference="${lr}_wheel">
-    <mu1 value="1.0" />
-    <mu2 value="1.0" />
+    <mu1 value="100.0" />
+    <mu2 value="100.0" />
     <kp value="10000000.0" />
     <kd value="1.0" />

Commit message: additional changes to planner params and sim environment

File: src/furiguide_description/urdf/furiguide.xacro (robot description, xacro)
@@ -12,5 +12,5 @@
 <xacro:property name="caster_height" value="0.04725" />
 <xacro:property name="caster_radius" value="0.020" />
-<xacro:property name="caster_offset" value="0.115" />
+<xacro:property name="caster_offset" value="0.115" />1
 <xacro:property name="caster_mass" value="0.5" />
 <xacro:property name="wheel_mass" value="1.0" />
@@ -38,7 +38,7 @@
       <origin xyz="0 0 0" />
       <inertia
-        ixx="0.01" ixy="0" ixz="0"
-        iyy="0.01" iyz="0"
-        izz="0.01"
+        ixx="0.001" ixy="0" ixz="0"
+        iyy="0.001" iyz="0"
+        izz="0.001"
       />
     </inertial>
